File: ESP-Easy FHEM Multi.brd (EAGLE design)
At the start: 37.8 x 63.7 mm, 26 parts, among them IC1 OKI-78SR-3.3, X1 MKDSN1,5/2-5,08, X2 MKDSN1,5/2-5,08, X3 MKDSN1,5/2-5,08

Commit message: Review Changes
Parts:
- moved R3 10.6 mm to (31.2, 26.2)
- moved JP3 8.64 mm to (25.9, 31.5)
- moved JP1 2.54 mm to (31.2, 31.5), turned to 90 degrees
- moved D5 1.27 mm to (18.8, 41.7)
- moved D6 1.27 mm to (12.2, 41.7)
- moved C1 0.76 mm to (23.6, 9.40)
Connections:
- net +3V3: now also JP2.11, JP2.13, JP2.9; no longer JP2.1, JP2.3, JP2.5
- net GND: now also JP2.1, JP2.3, JP2.5; no longer JP2.11, JP2.13, JP2.9
- net RESET: no longer S1.1
Routing:
- net +3V3: track 0.00 -> 83.2 mm
- net GND: track 39.3 -> 0.00 mm, vias 20 -> 16
- net RX: track 35.4 -> 25.1 mm
- net TX: track 36.0 -> 26.7 mm
- net GPIO0: track 21.8 -> 28.3 mm
- net RESET: track 47.7 -> 45.3 mm
- net +24V: track 62.6 -> 64.3 mm
- net GPIO14: track 12.5 -> 13.3 mm
- net GPIO5: track 35.8 -> 36.6 mm
- net N$2: track 13.9 -> 14.5 mm
- net N$3: track 15.8 -> 15.3 mm
- added copper zone on layer 1, net GND
- removed copper zone on layer 1, net +3V3
Other:
- board text added: "Flash"
- board text added: "GND"
- board text added: "RX"
- board text added: "TX"
- board text added: "UART"

Commit message: Last review changes
Parts:
- moved R1 3.36 mm to (29.4, 22.8), turned to 90 degrees
- moved X3 0.25 mm to (3.81, 45.2)
- moved X2 0.25 mm to (24.6, 59.9)
- moved R3 0.20 mm to (31.2, 26.0)
Connections:
- net +24V: now also X3.1; no longer X3.2
- net GND: now also X3.2; no longer X3.1
Routing:
- net +24V: track 64.3 -> 60.9 mm
- net +3V3: track 83.2 -> 82.0 mm
- net RESET: track 45.3 -> 46.1 mm
- added copper zone on layer 1, net N$4
Other:
- board text added: "Designed by: Sascha MzH"
- board text added: "ESP-Easy FHEM Multi"
- board text added: "v 1.0"
